File: Tinker shield/TinkerShieldPaddle/TinkerShieldPaddle.kicad_pcb (KiCad board)
At the start: 2 copper layers, 19.8 x 34.2 mm, 28 parts, among them J1 Batt, J2 Conn_01x05, J3 Audio-Jack-3, J4 Conn_01x02, J5 Conn_01x04, J6 Conn_01x04, Q1 2N7002, Q2 2N7002, U1 ADS1115IDGS, U2 MCP73831-2-OT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

Commit message: Add files via upload
Parts:
- removed ? (x4): , MountingHole:MountingHole_2.2mm_M2
- added R1: 10k, Resistor_SMD:R_0805_2012Metric_Pad1.15x1.40mm_HandSolder, F.Cu at (153.2, 145.2)
- added R3: 10k, Resistor_SMD:R_0805_2012Metric_Pad1.15x1.40mm_HandSolder, F.Cu at (165.2, 141.5)
- D1: value LED -> LED RED
- D2: value LED -> LED GREEN
- moved Q2 5.62 mm to (159.8, 129.2), turned to 180 degrees
- moved Q1 5.50 mm to (162.8, 124.5), turned to 90 degrees
Connections:
- Q1 pad 3: Net-(J3-Pad1) -> Net-(J3-Pad2)
- Q2 pad 3: Net-(J3-Pad2) -> Net-(J3-Pad1)
Routing:
- net Net-(C1-Pad2): track 38.6 -> 48.6 mm
- net GND: track 6.66 -> 14.7 mm
- net Net-(Q1-Pad1): track 24.7 -> 27.4 mm
- net Net-(Q2-Pad1): track 31.9 -> 30.6 mm
- net Net-(J3-Pad1): track 6.20 -> 5.36 mm

Commit message: Add files via upload
Parts:
- added REF**: MountingHole_2.2mm_M2_Pad, MountingHole:MountingHole_2.2mm_M2_Pad, F.Cu at (152.8, 120.5)
- added REF**: MountingHole_2.2mm_M2_Pad, MountingHole:MountingHole_2.2mm_M2_Pad, F.Cu at (167.5, 120.5)
- added REF**: MountingHole_2.2mm_M2_Pad, MountingHole:MountingHole_2.2mm_M2_Pad, F.Cu at (167.5, 149.8)
- added REF**: MountingHole_2.2mm_M2_Pad, MountingHole:MountingHole_2.2mm_M2_Pad, F.Cu at (152.8, 149.8)
Changed lines of the file:
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@@
     (tracks 170)
     (zones 0)
-    (modules 26)
+    (modules 30)
     (nets 25)
   )
@@
     (34 B.Paste user)
     (35 F.Paste user)
-    (36 B.SilkS user hide)
+    (36 B.SilkS user)
     (37 F.SilkS user)
     (38 B.Mask user)
@@
     (mod_text_size 1 1)
     (mod_text_width 0.15)
-    (pad_size 1.524 1.524)
-    (pad_drill 0.762)
+    (pad_size 4.4 4.4)
+    (pad_drill 2.2)
     (pad_to_mask_clearance 0.051)
     (solder_mask_min_width 0.25)
@@
     )
   )
+  (module MountingHole:MountingHole_2.2mm_M2_Pad (layer F.Cu)
+    (at 152.75 120.5)
+    (descr "Mounting Hole 2.2mm, M2")
+    (tags "mounting hole 2.2mm m2")
+    (attr virtual)
+    (fp_text reference REF** (at 0 -3.2) (layer F.SilkS)
+      (effects (font (size 1 1) (thickness 0.15)))
+    )
+    (fp_text value MountingHole_2.2mm_M2_Pad (at 0 3.2) (layer F.Fab)
+      (effects (font (size 1 1) (thickness 0.15)))
+    )
+    (fp_circle (center 0 0) (end 2.45 0) (layer F.CrtYd) (width 0.05))
+    (fp_circle (center 0 0) (end 2.2 0) (layer Cmts.User) (width 0.15))
+    (fp_text user %R (at 0.3 0) (layer F.Fab)
+      (effects (font (size 1 1) (thickness 0.15)))
+    )
+    (pad 1 thru_hole circle (at 0 0) (size 4.4 4.4) (drill 2.2) (layers *.Cu *.Mask)
+      (net 1 GND))
+  )
+  (module MountingHole:MountingHole_2.2mm_M2_Pad (layer F.Cu)
+    (at 167.5 120.5)
+    (descr "Mounting Hole 2.2mm, M2")
+    (tags "mounting hole 2.2mm m2")
+    (attr virtual)
+    (fp_text reference REF** (at 0 -3.2) (layer F.SilkS)
+      (effects (font (size 1 1) (thickness 0.15)))
+    )
+    (fp_text value MountingHole_2.2mm_M2_Pad (at 0 3.2) (layer F.Fab)
+      (effects (font (size 1 1) (thickness 0.15)))
+    )
+    (fp_circle (center 0 0) (end 2.45 0) (layer F.CrtYd) (width 0.05))
+    (fp_circle (center 0 0) (end 2.2 0) (layer Cmts.User) (width 0.15))
+    (fp_text user %R (at 0.3 0) (layer F.Fab)
+      (effects (font (size 1 1) (thickness 0.15)))
+    )
+    (pad 1 thru_hole circle (at 0 0) (size 4.4 4.4) (drill 2.2) (layers *.Cu *.Mask)
+      (net 1 GND))
+  )
+  (module MountingHole:MountingHole_2.2mm_M2_Pad (layer F.Cu)
+    (at 167.5 149.75)
+    (descr "Mounting Hole 2.2mm, M2")
+    (tags "mounting hole 2.2mm m2")
+    (attr virtual)
+    (fp_text reference REF** (at 0 -3.2) (layer F.SilkS)
+      (effects (font (size 1 1) (thickness 0.15)))
+    )
+    (fp_text value MountingHole_2.2mm_M2_Pad (at 0 3.2) (layer F.Fab)
+      (effects (font (size 1 1) (thickness 0.15)))
+    )
+    (fp_circle (center 0 0) (end 2.45 0) (layer F.CrtYd) (width 0.05))
+    (fp_circle (center 0 0) (end 2.2 0) (layer Cmts.User) (width 0.15))
+    (fp_text user %R (at 0.3 0) (layer F.Fab)
+      (effects (font (size 1 1) (thickness 0.15)))
+    )
+    (pad 1 thru_hole circle (at 0 0) (size 4.4 4.4) (drill 2.2) (layers *.Cu *.Mask)
+      (net 1 GND))
+  )
+  (module MountingHole:MountingHole_2.2mm_M2_Pad (layer F.Cu)
+    (at 152.75 149.75)
+    (descr "Mounting Hole 2.2mm, M2")
+    (tags "mounting hole 2.2mm m2")
+    (attr virtual)
+    (fp_text reference REF** (at 0 -3.2) (layer F.SilkS)
+      (effects (font (size 1 1) (thickness 0.15)))
+    )
+    (fp_text value MountingHole_2.2mm_M2_Pad (at 0 3.2) (layer F.Fab)
+      (effects (font (size 1 1) (thickness 0.15)))
+    )
+    (fp_circle (center 0 0) (end 2.45 0) (layer F.CrtYd) (width 0.05))
+    (fp_circle (center 0 0) (end 2.2 0) (layer Cmts.User) (width 0.15))
+    (fp_text user %R (at 0.3 0) (layer F.Fab)
+      (effects (font (size 1 1) (thickness 0.15)))
+    )
+    (pad 1 thru_hole circle (at 0 0) (size 4.4 4.4) (drill 2.2) (layers *.Cu *.Mask)
+      (net 1 GND))
+  )
   (gr_line (start 170 152.25) (end 170 149.75) (layer Edge.Cuts) (width 0.15))
