File: Tinker shield/TinkerShieldPaddle/TinkerShieldPaddle.kicad_pcb (KiCad board)
At the start: 2 copper layers, 19.8 x 34.2 mm, 30 parts, among them J1 Batt, J2 Conn_01x05, J3 Audio-Jack-3, J4 Conn_01x02, J5 Conn_01x04, J6 Conn_01x04, Q1 2N7002, Q2 2N7002, U1 ADS1115IDGS, U2 MCP73831-2-OT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

Commit message: Add files via upload
Routing:
- net GND: track 14.7 -> 36.8 mm
Changed lines of the file:
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@@
     (thickness 1.6)
     (drawings 12)
-    (tracks 170)
+    (tracks 186)
     (zones 0)
     (modules 30)
@@
   (gr_line (start 170 118) (end 170 149.75) (layer Edge.Cuts) (width 0.15))
   (segment (start 155.5 141.35) (end 155.75 141.1) (width 0.25) (layer F.Cu) (net 1))
-  (segment (start 155.5 142.15) (end 155.5 141.35) (width 0.25) (layer F.Cu) (net 1))
   (segment (start 157.376628 141.401628) (end 158 142.025) (width 0.25) (layer F.Cu) (net 1))
   (segment (start 157.202028 141.401628) (end 157.376628 141.401628) (width 0.25) (layer F.Cu) (net 1))
@@
   (segment (start 155.5 143.5) (end 155.25 143.75) (width 0.25) (layer F.Cu) (net 1))
   (segment (start 152.68681 145.25) (end 151.5 144.06319) (width 0.25) (layer F.Cu) (net 1))
+  (segment (start 162.549999 142.100001) (end 162.549999 141.436411) (width 0.25) (layer F.Cu) (net 1))
+  (segment (start 162.5 142.15) (end 162.549999 142.100001) (width 0.25) (layer F.Cu) (net 1))
+  (segment (start 162.549999 141.436411) (end 162.98641 141) (width 0.25) (layer F.Cu) (net 1))
+  (segment (start 162.98641 141) (end 163.75 141) (width 0.25) (layer F.Cu) (net 1))
+  (segment (start 156.934001 141.274999) (end 155.575001 141.274999) (width 0.25) (layer F.Cu) (net 1))
+  (segment (start 155.5 141.35) (end 155.5 142.15) (width 0.25) (layer F.Cu) (net 1))
+  (segment (start 159.845001 144.185999) (end 156.934001 141.274999) (width 0.25) (layer F.Cu) (net 1))
+  (segment (start 159.845001 145.314001) (end 159.845001 144.185999) (width 0.25) (layer F.Cu) (net 1))
+  (segment (start 166.13499 143.921798) (end 166.13499 146.0786) (width 0.25) (layer F.Cu) (net 1))
+  (segment (start 165.788191 143.574999) (end 166.13499 143.921798) (width 0.25) (layer F.Cu) (net 1))
+  (segment (start 155.575001 141.274999) (end 155.5 141.35) (width 0.25) (layer F.Cu) (net 1))
+  (segment (start 164.711809 143.574999) (end 165.788191 143.574999) (width 0.25) (layer F.Cu) (net 1))
+  (segment (start 164.22499 143.08818) (end 164.711809 143.574999) (width 0.25) (layer F.Cu) (net 1))
+  (segment (start 160.6096 146.0786) (end 159.845001 145.314001) (width 0.25) (layer F.Cu) (net 1))
+  (segment (start 164.22499 141.47499) (end 164.22499 143.08818) (width 0.25) (layer F.Cu) (net 1))
+  (segment (start 166.13499 146.0786) (end 160.6096 146.0786) (width 0.25) (layer F.Cu) (net 1))
+  (segment (start 163.75 141) (end 164.22499 141.47499) (width 0.25) (layer F.Cu) (net 1))
   (segment (start 158.5 144.58) (end 158.67 144.75) (width 0.25) (layer F.Cu) (net 2))
   (segment (start 157.820001 143.900001) (end 158.67 144.75) (width 0.25) (layer F.Cu) (net 2))
